File: LampBoard.sch (EAGLE design)
At the start: 28 parts, among them IC1 MEGA8-AI, J1 70543-04, J2 70543-05, T1 BTA25

Commit message: Procesor moved away from Power board
Parts:
- removed IC1: MEGA8-AI, atmel:MEGA8-AI
- removed ISP1: AVRISP-BOX, adafruit:AVRISP-BOX
- removed J1: 70543-04, con-molex-c-grid:70543-04
- removed J2: 70543-05, con-molex-c-grid:70543-05
- removed LED3, LED4: (no value), led:LED3MM
- removed R6, R7: (no value), rcl:R-EU_R0805
- added X1: HEADER_POS4_70543, con-molex-c-grid-sl:HEADER_POS4_70543
- R1, R8: value 1M -> 22k
- R3: value 100R -> 22k
- R4: value (none) -> 1k; device rcl:R-EU_R0805 -> rcl:R-EU_M0805
Connections:
- removed net IRQ: IC1.PC3(ADC3), J2.2
- removed net MISO: IC1.PB4(MISO), ISP1.MISO
- removed net MOSI: IC1.PB3(MOSI/OC2), ISP1.MOSI
- removed net N$10: IC1.PD7(AIN1), LED3.A
- removed net N$13: IC1.PD6(AIN0), LED4.A
- removed net N$14: LED4.C, R6.2
- removed net N$15: LED3.C, R7.2
- removed net RESET: IC1.PC6(/RESET), ISP1.RST, R4.1
- removed net RXD: IC1.PD0(RXD), J1.2
- removed net SCK: IC1.PB5(SCK), ISP1.SCK
- removed net SCL: IC1.PC5(ADC5/SCL), J2.4
- removed net SDA: IC1.PC4(ADC4/SDA), J2.3
- removed net TXD: IC1.PD1(TXD), J1.3
- net +5V: now also X1.4; no longer IC1.AVCC, IC1.VCC@1, IC1.VCC@2, ISP1.VCC, J1.1, J2.1
- net GND: now also X1.3; no longer IC1.GND, IC1.GND@1, IC1.GND@2, ISP1.GND, J1.4, J2.5, R6.1, R7.1
- net SWITCH: now also X1.1; no longer IC1.PD2(INT0)
- net ZERO: now also R4.1, X1.2; no longer IC1.PD3(INT1)
Other:
- moved on the sheet: R4
